File: KiCad/DC_to_DC_Converter/ISL6236AIRZ/ISL6236AIRZ.kicad_sch (KiCad schematic)
At the start: 0 parts

Commit message: added symbols to the schematic
Parts:
- added C1, C2: 1uF, symbol custom_symbol_library:CAP0805 X7R 1UF
- added C3: 0.01uF, symbol custom_symbol_library:0.01_µF_Ceramic_Capacitor
- added C4: 0.1uF, symbol custom_symbol_library:Capacitor_X7R_0805_0.1uF
- added R1, R2, R3, R4: 200k, symbol custom_symbol_library:RES_200K_OHM
- added U1: ISL6236A, symbol custom_symbol_library:ISL6236AIRZ
- added U2, U3: SI4816BDY, symbol custom_symbol_library:SI4816BDY
Connections:
- new net: C4.1, U1.1 (REF)
- new net: R2.1, U1.31 (ILIM2)
- new net: U1.26 (UGATE2), U2.1 (G1)
- new net: U1.23 (LGATE2), U2.4 (D1)
- new net: C2.1, U1.3 (VCC)
- new net: R3.2, U1.13 (POK1)
- new net: C3.1, U1.5 (VREF3)
- new net: R1.2, U1.12 (ILIM1)
- new net: U1.15 (UGATE1), U3.1 (G1)
- new net: U1.18 (LGATE1), U3.4 (D1)
- new net: R4.2, U1.28 (POK2)
- new net +5V: C1.2, R3.1, R4.1, U1.19 (PVCC)
- new net GND: C1.1, C2.2, C3.2, C4.2, R1.1, R2.2, U1.21 (GND), U1.29 (~{SKIP}), U1.33 (EP)
